Commit message: Update files

File: urdf/cylinder.xacro (robot description, xacro)
@@ -1,3 +1,8 @@
+<?xml version="1.0"?>
 <robot name="cylinder" xmlns:xacro="http://ros.org/wiki/xacro">
+ <!-- Define robot constants -->
+ <xacro:property name="base_radius" value="0.12"/>
+ <xacro:property name="base_length" value="0.093"/>
+ <!-- Robot Base -->
  <link name="base_link">
   <inertial>
@@ -8,5 +13,5 @@
   <visual>
    <geometry>
-    <cylinder length="0.093" radius="0.12"/>
+    <cylinder length="${base_length}" radius="${base_radius}"/>
    </geometry>
    <material name="blue">
@@ -16,5 +21,5 @@
   <collision>
    <geometry>
-    <cylinder length="0.093" radius="0.12"/>
+    <cylinder length="${base_length}" radius="${base_radius}"/>
    </geometry>
   </collision>

File: urdf/cylinder_gazebo.xacro (robot description, xacro)
@@ -1,2 +1,3 @@
+<?xml version="1.0"?>
 <robot name="cylinder" xmlns:xacro="http://ros.org/wiki/xacro">
  <link name="base_link" />
